File: BatteryChecker.kicad_pcb (KiCad board)
At the start: 2 copper layers, 52.1 x 86.4 mm, 43 parts, among them J1 USB_B_Micro, Q1 PN2222A, U1 LM358, U2 LM358

Commit message: Updated v3.0
Parts:
- removed the ? at (92.7, 101.6) (x2)
- removed Q1: PN2222A, Package_TO_SOT_THT:TO-92_Inline_Wide
- removed R14: 1kohm, Resistor_THT:R_Axial_DIN0207_L6.3mm_D2.5mm_P10.16mm_Horizontal
- added ? (x2): , , F.Cu at (92.7, 101.6)
- added J2: Conn_02x02, Connector_PinHeader_1.27mm:PinHeader_2x02_P1.27mm_Vertical, F.Cu at (90.2, 67.3)
- moved R4 10.2 mm to (92.7, 76.2), turned to 180 degrees
- moved R5 10.2 mm to (82.5, 80.0), turned to 0 degrees
- moved R9 10.2 mm to (82.5, 83.8), turned to 0 degrees
- moved D6 4.02 mm to (109.2, 94.0), turned to 90 degrees
- moved R10 1.27 mm to (102.9, 101.6)
- moved R11 1.27 mm to (102.9, 115.6)
- moved R12 1.27 mm to (102.9, 129.5)
- moved R13 1.27 mm to (102.9, 143.5)
- turned D1 to 180 degrees
- turned D2 to 180 degrees
- turned D3 to 180 degrees
- turned D4 to 180 degrees
- turned D5 to 180 degrees
Connections:
- D1 pad 2: Net-(D1-Pad2) -> R
- D6 pad 1: Net-(D6-Pad1) -> R
- R4 pad 2: Net-(R4-Pad2) -> Net-(J2-Pad2)
- R5 pad 1: Net-(R4-Pad2) -> Net-(J2-Pad2)
- R9 pad 1: Net-(D1-Pad2) -> R
- U1 pad 2: Net-(R4-Pad2) -> Net-(J2-Pad3)
- U1 pad 3: TEST -> Net-(J2-Pad4)
Routing:
- net Net-(D1-Pad2): track 52.6 -> 0.00 mm
- net R: track 0.00 -> 36.5 mm
- net Net-(R4-Pad2): track 26.5 -> 0.00 mm
- net Net-(R5-Pad2): track 40.5 -> 16.9 mm
- net Net-(D6-Pad1): track 20.6 -> 0.00 mm
- net Net-(J2-Pad2): track 0.00 -> 19.9 mm
- net +5V: track 151.6 -> 135.8 mm
- net Net-(D4-Pad2): track 13.5 -> 5.08 mm
- net Net-(J2-Pad4): track 0.00 -> 5.61 mm
- net Net-(D5-Pad2): track 12.0 -> 6.66 mm
- net Net-(D3-Pad2): track 12.0 -> 6.66 mm
- net G: track 29.8 -> 25.5 mm
- net Net-(R9-Pad2): track 26.1 -> 22.4 mm
- net Net-(J2-Pad3): track 0.00 -> 3.34 mm
- net TEST: track 101.2 -> 98.3 mm
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Other:
- board size 52.1 x 86.4 mm -> 48.3 x 86.4 mm
- board text added: "+ -"
- board text added: "2022-01-09 v3.0"
- board text added: "9V"
- board text added: "Battery Checker v3 Christoffer Karlsson"
- board text removed: "2022-01-08 v2.0"
- board text removed: "9V + -"
- board text removed: "Battery Checker v2 Christoffer Karlsson 2022"

Commit message: Updated PCB and schematic
Parts:
- removed the ? at (92.7, 101.6) (x2)
- added ? (x2): , , F.Cu at (92.7, 101.6)
- moved D3 1.27 mm to (110.5, 120.7)
- moved D4 1.27 mm to (110.5, 130.8)
- moved D5 1.27 mm to (110.5, 141.0)
- moved D1 1.27 mm to (110.5, 100.3)
- moved D2 1.27 mm to (110.5, 110.5)
Routing:
- net R: track 36.5 -> 37.8 mm
- net G: track 25.5 -> 26.8 mm
- net Net-(D5-Pad2): track 6.66 -> 6.13 mm
- net Net-(D4-Pad2): track 5.08 -> 5.61 mm
- net Net-(D3-Pad2): track 6.66 -> 7.18 mm
Other:
- board text added: "2022-01-11 v3.0"
- board text removed: "2022-01-09 v3.0"
