File: BatteryChecker.sch (KiCad schematic (older format))
At the start: 40 parts, among them J1 USB_B_Micro, Q1 PN2222A, U1 LM358, U2 LM358

Commit message: Updated v3.0
Parts:
- removed Q1: PN2222A, Package_TO_SOT_THT:TO-92_Inline_Wide, symbol Transistor_BJT:PN2222A
- removed R14: 1kohm, Resistor_THT:R_Axial_DIN0207_L6.3mm_D2.5mm_P10.16mm_Horizontal, symbol Device:R_US
- added J2: Mode selector, Connector_PinHeader_1.27mm:PinHeader_2x02_P1.27mm_Vertical, symbol Connector_Generic:Conn_02x02_Counter_Clockwise
Connections:
- net TEST: now also J2.1 (Pin_1); no longer U1.3 (+)
- net at R4.2, R5.1: now also J2.2 (Pin_2); no longer U1.2 (-)
- net R: now reaches D6.1 (RA)
- net R: now also D1.2 (A), R9.1
- new net: J2.3 (Pin_3), U1.2 (-)
- new net: J2.4 (Pin_4), U1.3 (+)
Other:
- moved on the sheet: D6, R4, R5, R6, R7, R8
